Commit message: all working uptill corridor env, heading command is sus, backup for local breakdown

File: humanoid/envs/navi/man.urdf (robot description, URDF)
Before this commit: robot object, 1 links, 0 joints
Links:
- link object: geometry collision box size=0.42 0.42 1; visual mesh filename=woman.obj scale=.0077 .0077 .0077

Commit message: heading working, corridor env finished, time to start grinding demos

File: humanoid/envs/navi/man.urdf (robot description, URDF)
Before this commit: robot object, 1 links, 0 joints
Links:
- link object: geometry collision box size=0.42 0.42 1; visual mesh filename=woman.obj scale=.0096 .0096 .0096
